Commit message: 16/07/2024 23:07

File: paquete_proyecto/urdf/proyecto_xacro.urdf (robot description, URDF)
Before this commit: robot robot_name, 4 links, 3 joints
Links:
- link antebrazo: mass 0.01 -> None; geometry collision box size=${lado_caja_antebrazo} ${lado_caja_antebrazo} ${alto_caja_a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; visual box size=${lado_caja_antebrazo} ${lado_caja_antebrazo} ${alto_caja_a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
- link base_giratoria: mass 0.01 -> None; geometry collision cylinder length=${alto_cilindro} radius=${radio_cilindro}; visual cylinder length=${alto_cilindro} radius=${radio_cilindro}
- link base_link: mass 50 -> None; geometry collision box size=${lado_caja_base} ${lado_caja_base} ${alto_caja_base}; visual box size=${lado_caja_base} ${lado_caja_base} ${alto_caja_base}
- link brazo: mass 0.01 -> None; geometry collision box size=${lado_caja_brazo} ${lado_caja_brazo} ${alto_caja_brazo}; visual box size=${lado_caja_brazo} ${lado_caja_brazo} ${alto_caja_brazo}
Joints:
- joint antebrazo_brazo_joint: limit lower=0 upper=2.6927937030769655 effort=100 velocity=100 -> lower=0 upper=${pi} effort=100 velocity=100; origin xyz=0.0 0.0 0.4 rpy=0.0 0.0 0.0 -> xyz=0.0 0.0 ${alto_caja_brazo} rpy=0.0 0.0 0.0
- joint base_brazo_joint: limit lower=-1.5707963267948966 upper=1.5707963267948966 effort=100 velocity=100 -> lower=0 upper=${pi/2} effort=100 velocity=100; origin xyz=0.0 0.0 0.05 rpy=0.0 0.0 0.0 -> xyz=0.0 ${-lado_caja_brazo/2} ${alto_cilindro} rpy=0.0 0.0 0.0
- joint base_giro_joint: limit lower=-1.5707963267948966 upper=1.5707963267948966 effort=100 velocity=100 -> lower=${-pi/2} upper=${pi/2} effort=100 velocity=100; origin xyz=0.0 0.0 0.1 rpy=0.0 0.0 0.0 -> xyz=0.0 0.0 ${alto_caja_base} rpy=0.0 0.0 0.0
